Commit message: Update sensor model

File: sensor_kit/e1r_sensor_kit_launch/e1r_sensor_kit_description/urdf/sensor_kit.xacro (robot description, xacro)
@@ -50,5 +50,5 @@
       />
     </xacro:VLP-16>
-    <!-- camera -->
+    camera
     <xacro:monocular_camera_macro
       name="traffic_light_right_camera/camera"
@@ -171,5 +171,5 @@
       fov="1.3"
     />
-    <!-- gnss -->
+    gnss
     <xacro:imu_macro
       name="gnss"
@@ -184,5 +184,5 @@
       fps="100"
     />
-    <!-- imu -->
+    imu
     <xacro:imu_macro
       name="tamagawa/imu"
@@ -196,5 +196,5 @@
       yaw="${calibration['sensor_kit_base_link']['tamagawa/imu_link']['yaw']}"
       fps="100"
-    />
-  </xacro:macro> -->
+    /> -->
+  </xacro:macro>
 </robot>

Commit message: Add new e1r sensor kit

File: sensor_kit/e1r_sensor_kit_launch/e1r_sensor_kit_description/urdf/sensor_kit.xacro (robot description, xacro)
@@ -22,34 +22,14 @@
     <xacro:VLS-128 parent="sensor_kit_base_link" name="rslidar" topic="/rs_lidar/points" hz="10" samples="220" gpu="$(arg gpu)">
       <origin
-        xyz="${calibration['sensor_kit_base_link']['rslidar']['x']}
-             ${calibration['sensor_kit_base_link']['rslidar']['y']}
-             ${calibration['sensor_kit_base_link']['rslidar']['z']}"
-        rpy="${calibration['sensor_kit_base_link']['rslidar']['roll']}
-             ${calibration['sensor_kit_base_link']['rslidar']['pitch']}
-             ${calibration['sensor_kit_base_link']['rslidar']['yaw']}"
+        xyz="${calibration['sensor_kit_base_link']['rslidar_base_link']['x']}
+             ${calibration['sensor_kit_base_link']['rslidar_base_link']['y']}
+             ${calibration['sensor_kit_base_link']['rslidar_base_link']['z']}"
+        rpy="${calibration['sensor_kit_base_link']['rslidar_base_link']['roll']}
+             ${calibration['sensor_kit_base_link']['rslidar_base_link']['pitch']}
+             ${calibration['sensor_kit_base_link']['rslidar_base_link']['yaw']}"
       />
     </xacro:VLS-128>
-    <!-- <xacro:VLP-16 parent="sensor_kit_base_link" name="velodyne_left" topic="/points_raw" hz="10" samples="220" gpu="$(arg gpu)">
-      <origin
-        xyz="${calibration['sensor_kit_base_link']['velodyne_left_base_link']['x']}
-             ${calibration['sensor_kit_base_link']['velodyne_left_base_link']['y']}
-             ${calibration['sensor_kit_base_link']['velodyne_left_base_link']['z']}"
-        rpy="${calibration['sensor_kit_base_link']['velodyne_left_base_link']['roll']}
-             ${calibration['sensor_kit_base_link']['velodyne_left_base_link']['pitch']}
-             ${calibration['sensor_kit_base_link']['velodyne_left_base_link']['yaw']}"
-      />
-    </xacro:VLP-16>
-    <xacro:VLP-16 parent="sensor_kit_base_link" name="velodyne_right" topic="/points_raw" hz="10" samples="220" gpu="$(arg gpu)">
-      <origin
-        xyz="${calibration['sensor_kit_base_link']['velodyne_right_base_link']['x']}
-             ${calibration['sensor_kit_base_link']['velodyne_right_base_link']['y']}
-             ${calibration['sensor_kit_base_link']['velodyne_right_base_link']['z']}"
-        rpy="${calibration['sensor_kit_base_link']['velodyne_right_base_link']['roll']}
-             ${calibration['sensor_kit_base_link']['velodyne_right_base_link']['pitch']}
-             ${calibration['sensor_kit_base_link']['velodyne_right_base_link']['yaw']}"
-      />
-    </xacro:VLP-16>
-    camera
-    <xacro:monocular_camera_macro
+    <!-- camera -->
+    <!-- <xacro:monocular_camera_macro
       name="traffic_light_right_camera/camera"
       parent="sensor_kit_base_link"
@@ -170,6 +150,6 @@
       height="400"
       fov="1.3"
-    />
-    gnss
+    /> -->
+    <!-- gnss -->
     <xacro:imu_macro
       name="gnss"
@@ -184,6 +164,6 @@
       fps="100"
     />
-    imu
-    <xacro:imu_macro
+    <!-- imu -->
+    <!-- <xacro:imu_macro
       name="tamagawa/imu"
       parent="sensor_kit_base_link"

File: sensor_kit/e1r_sensor_kit_launch/e1r_sensor_kit_description/urdf/sensors.xacro (robot description, xacro)
@@ -14,6 +14,6 @@
     yaw="${calibration['base_link']['sensor_kit_base_link']['yaw']}"
   />
-  <!-- embedded sensors
-  <xacro:include filename="$(find velodyne_description)/urdf/VLP-16.urdf.xacro"/>
+  <!-- embedded sensors -->
+  <!-- <xacro:include filename="$(find velodyne_description)/urdf/VLP-16.urdf.xacro"/>
   <xacro:VLP-16 parent="base_link" name="velodyne_rear" topic="velodyne_rear/velodyne_points" hz="10" samples="220" gpu="false">
     <origin

Commit message: Add XSens gnss and imu

File: sensor_kit/e1r_sensor_kit_launch/e1r_sensor_kit_description/urdf/sensor_kit.xacro (robot description, xacro)
@@ -30,5 +30,5 @@
       />
     </xacro:VLS-128>
-    <!-- gnss -->
+    <!-- gnss + imu -->
     <xacro:imu_macro
       name="imu"
@@ -43,15 +43,4 @@
       fps="100"
     />
-    <!-- imu -->
-    <xacro:VLS-128 parent="sensor_kit_base_link" name="rslidar" topic="/rs_imu" hz="10" samples="220" gpu="$(arg gpu)">
-      <origin
-        xyz="${calibration['sensor_kit_base_link']['rslidar_base_link']['x']}
-             ${calibration['sensor_kit_base_link']['rslidar_base_link']['y']}
-             ${calibration['sensor_kit_base_link']['rslidar_base_link']['z']}"
-        rpy="${calibration['sensor_kit_base_link']['rslidar_base_link']['roll']}
-             ${calibration['sensor_kit_base_link']['rslidar_base_link']['pitch']}
-             ${calibration['sensor_kit_base_link']['rslidar_base_link']['yaw']}"
-      />
-    </xacro:VLS-128>
     <!-- camera -->
     <!-- <xacro:monocular_camera_macro

Commit message: gyro_odom with ac1 - provision for eagleye using multiantenna

File: sensor_kit/e1r_sensor_kit_launch/e1r_sensor_kit_description/urdf/sensor_kit.xacro (robot description, xacro)
@@ -19,6 +19,28 @@
     <!-- sensor -->
     <xacro:property name="calibration" value="${xacro.load_yaml('$(arg config_dir)/sensor_kit_calibration.yaml')}"/>
+    <!-- lidar
+    <xacro:VLS-128 parent="sensor_kit_base_link" name="e1rlidar" topic="/e1r_lidar_points" hz="10" samples="220" gpu="$(arg gpu)">
+      <origin
+        xyz="${calibration['sensor_kit_base_link']['e1rlidar_base_link']['x']}
+             ${calibration['sensor_kit_base_link']['e1rlidar_base_link']['y']}
+             ${calibration['sensor_kit_base_link']['e1rlidar_base_link']['z']}"
+        rpy="${calibration['sensor_kit_base_link']['e1rlidar_base_link']['roll']}
+             ${calibration['sensor_kit_base_link']['e1rlidar_base_link']['pitch']}
+             ${calibration['sensor_kit_base_link']['e1rlidar_base_link']['yaw']}"
+      />
+    </xacro:VLS-128> -->
     <!-- lidar -->
-    <xacro:VLS-128 parent="sensor_kit_base_link" name="e1rlidar" topic="/e1r_lidar_points" hz="10" samples="220" gpu="$(arg gpu)">
+    <xacro:VLS-128 parent="sensor_kit_base_link" name="rslidar" topic="/sensing/lidar/pointcloud_raw_ex" hz="10" samples="220" gpu="$(arg gpu)">
+      <origin
+        xyz="${calibration['sensor_kit_base_link']['rslidar_base_link']['x']}
+             ${calibration['sensor_kit_base_link']['rslidar_base_link']['y']}
+             ${calibration['sensor_kit_base_link']['rslidar_base_link']['z']}"
+        rpy="${calibration['sensor_kit_base_link']['rslidar_base_link']['roll']}
+             ${calibration['sensor_kit_base_link']['rslidar_base_link']['pitch']}
+             ${calibration['sensor_kit_base_link']['rslidar_base_link']['yaw']}"
+      />
+    </xacro:VLS-128>
+    <!-- lidar -->
+    <xacro:VLS-128 parent="sensor_kit_base_link" name="e1rlidar" topic="/sensing/lidar/pointcloud_raw_ex" hz="10" samples="220" gpu="$(arg gpu)">
       <origin
         xyz="${calibration['sensor_kit_base_link']['e1rlidar_base_link']['x']}
