Commit message: Debugging.

File: sensor_kit/ac1_sensor_kit_launch/ac1_sensor_kit_description/urdf/sensor_kit.xacro (robot description, xacro)
@@ -70,3 +70,4 @@
       fps="100"
     />
+  </xacro:macro>
 </robot>

File: sensor_kit/ac1_sensor_kit_launch/ac1_sensor_kit_description/urdf/sensors.xacro (robot description, xacro)
@@ -14,4 +14,3 @@
     yaw="${calibration['base_link']['sensor_kit_base_link']['yaw']}"
   />
-  </xacro:VLP-16>
 </robot>

File: sensor_kit/e1r_sensor_kit_launch/e1r_sensor_kit_description/urdf/sensor_kit.xacro (robot description, xacro)
@@ -70,3 +70,4 @@
       fps="100"
     />
+  </xacro:macro>
 </robot>

File: sensor_kit/e1r_sensor_kit_launch/e1r_sensor_kit_description/urdf/sensors.xacro (robot description, xacro)
@@ -14,4 +14,3 @@
     yaw="${calibration['base_link']['sensor_kit_base_link']['yaw']}"
   />
-  </xacro:VLP-16>
 </robot>
